File: USB2UART_PROG/USB2UART_PROG.kicad_pcb (KiCad board)
At the start: 4 copper layers, 19 x 40 mm, 43 parts, among them J1 USB4105, J2 UART Header, J3 TC2030, SW1 BOOT, SW2 EN, U1 FT230, U2 USBLC6, U3 TLV1117

Commit message: BOOT & RESET ISSUE
Fixed a wrong connection with B&R buttons.
Parts:
- added kibuzzard-676ADB76: G***, kibuzzard-676ADB76, F.Cu at (134.5, 73.7)
- added kibuzzard-676ADB82: G***, kibuzzard-676ADB82, F.Cu at (134.5, 77.1)
Routing:
- net +3V3: track 31.6 -> 69.7 mm, vias 5 -> 7
- added copper zone on In2.Cu, net (none)
